File: zxIDE.kicad_pcb (KiCad board)
At the start: 2 copper layers, 5 parts, among them J1 Conn_02x20_Odd_Even, Q1 BC327, U1 74LS10, U2 Z80CPU

Commit message: add schematics in pdf and some pictures
Routing:
- net Net-(U1-Pad12): track 0.00 -> 9.12 mm
