File: zxIDE.sch (KiCad schematic (older format))
At the start: 5 parts, among them J1 Conn_02x20_Odd_Even, Q1 BC327, U1 74LS10, U2 Z80CPU

Commit message: add schematics in pdf and some pictures
Other:
- note added: "27/11/20"
- note added: "TurBo ZxIDE v0.1"
- note added: "TurBoss"
- note added: "ZX Spectrum 128K 2+ 8bit IDE"
- note added: "ZxIDE"
- moved on the sheet: J1, Q1, R1, U1A, U1B, U1C, U1D, U2
